File: schematics/fpgaboard/fpgaboard/RAM.kicad_sch (KiCad schematic)
At the start: 2 parts, among them U3 IS42S16320F-7TL, U4 IS42S16320F-7TL

Commit message: Work on connecting up SDRAM to FPGA.
Parts:
- added C10, C11, C8, C9: C_Small, Capacitor_SMD:C_0402_1005Metric, symbol Device:C_Small
Connections:
- net IO_3v3: now reaches U3.1 (VDD), U3.14 (VDD), U3.27 (VDD)
- net IO_3v3: now also U3.3 (VDDQ), U3.43 (VDDQ), U3.49 (VDDQ), U3.9 (VDDQ), U4.1 (VDD), U4.14 (VDD), U4.27 (VDD), U4.3 (VDDQ), U4.43 (VDDQ), U4.49 (VDDQ), U4.9 (VDDQ), C10.1, C11.1, C8.1, C9.1
- net GND: now reaches U3.12 (VSSQ), U3.46 (VSSQ), U3.52 (VSSQ), U3.6 (VSSQ)
- net GND: now also U3.28 (VSS), U3.41 (VSS), U3.54 (VSS), U4.12 (VSSQ), U4.28 (VSS), U4.41 (VSS), U4.46 (VSSQ), U4.52 (VSSQ), U4.54 (VSS), U4.6 (VSSQ), C10.2, C11.2, C8.2, C9.2
